File: hardware/switchModule/switch.kicad_sch (KiCad schematic)
At the start: 66 parts, among them J1 Button-Sensors-MicroMatch2X03, J10 Conn_01x06_Female, J11 Conn_01x06_Female, J12 SWITCHES-SENSORS, J2 Screw_Terminal_01x02, J5 IRDA, J6 IRDA, J7 RJ45-CAN, J8 Conn_01x06_Female, J9 Conn_01x06_Female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

Commit message: feat: change PCB debug to EN/BOOT0
Parts:
- removed J12: SWITCHES-SENSORS, awesome:02x03MicroMatch, symbol Connector:Conn_01x06_Female
- removed Q1, Q2: BC847, Package_TO_SOT_SMD:SOT-23, symbol Transistor_BJT:BC847
- removed R1, R2, R3: 10K, Resistor_SMD:R_0603_1608Metric_Pad0.98x0.95mm_HandSolder, symbol Device:R
- added J3: Button-Sensors-MicroMatch2X03, awesome:02x03MicroMatch, symbol awesome:Button-Sensors-MicroMatch2X03
- added R5, R6: 2K2, Resistor_SMD:R_0603_1608Metric_Pad0.98x0.95mm_HandSolder, symbol Device:R
Connections:
- net DTR is gone; now on net BOOT0: U6.6 (BOOT0)
- net RTS is gone; now on net EN: U6.1 (EN)
- net +3V3: now also J1.1 (VCC), J3.1 (VCC), R5.1, R6.1; no longer J1.6 (VCC)
- net GND: now also J1.6 (GND), J3.6 (GND); no longer J1.1 (GND)
- net SCL: now also J1.3 (B2/SCL), R6.2; no longer J1.4 (B2/SCL)
- net SDA: now also J1.2 (B1/SDA), R5.2; no longer J1.5 (B1/SDA)
- net SW1: now also J3.2 (B1/SDA)
- net SW2: now also J3.3 (B2/SCL)
- net SW3: now also J3.4 (B3)
- net SW4: now also J3.5 (B4)
- net at R16.2: now also J1.5 (B4); no longer J1.2 (B4)
- net at R17.2: now also J1.4 (B3); no longer J1.3 (B3)
