File: hardware/switchModule/switch.kicad_pcb (KiCad board)
At the start: 2 copper layers, 48 x 49 mm, 70 parts, among them J1 Button-Sensors-MicroMatch2X03, J10 Conn_01x06_Female, J11 Conn_01x06_Female, J12 SWITCHES-SENSORS, J2 Screw_Terminal_01x02, J5 IRDA, J6 IRDA, J7 RJ45-CAN, J8 Conn_01x06_Female, J9 Conn_01x06_Female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

Commit message: feat: change PCB debug to EN/BOOT0
Parts:
- removed J12: SWITCHES-SENSORS, awesome:02x03MicroMatch
- removed Q1, Q2: BC847, Package_TO_SOT_SMD:SOT-23
- removed R1, R2, R3: 10K, Resistor_SMD:R_0603_1608Metric_Pad0.98x0.95mm_HandSolder
- added J3: Button-Sensors-MicroMatch2X03, awesome:02x03MicroMatch, F.Cu at (101.5, 90.3)
- added R5: 2K2, Resistor_SMD:R_0603_1608Metric_Pad0.98x0.95mm_HandSolder, B.Cu at (114.8, 85.9)
- added R6: 2K2, Resistor_SMD:R_0603_1608Metric_Pad0.98x0.95mm_HandSolder, B.Cu at (117.4, 88.0)
- moved J1 6.03 mm to (117.4, 90.3), turned to 90 degrees
- moved C2 5.12 mm to (124.5, 86.0), turned to 180 degrees
- moved R4 4.48 mm to (124.5, 87.8)
Connections:
- J1 pad 1: GND -> +3V3
- J1 pad 2: Net-(J1-Pad2) -> /SDA
- J1 pad 3: Net-(J1-Pad3) -> /SCL
- J1 pad 4: /SCL -> Net-(J1-Pad4)
- J1 pad 5: /SDA -> Net-(J1-Pad5)
- J1 pad 6: +3V3 -> GND
- R16 pad 2: Net-(J1-Pad2) -> Net-(J1-Pad5)
- R17 pad 2: Net-(J1-Pad3) -> Net-(J1-Pad4)
- U6 pad 1: /RTS -> /EN
- U6 pad 6: /DTR -> /BOOT0
Routing:
- net /RTS: track 27.5 -> 0.00 mm
- net /DTR: track 13.8 -> 0.00 mm
- net Net-(J1-Pad5): track 0.00 -> 11.2 mm, vias 0 -> 1
- net Net-(J1-Pad2): track 11.1 -> 0.00 mm, vias 1 -> 0
- net /EN: track 53.4 -> 59.6 mm, vias 2 -> 3
- net /BOOT0: track 17.6 -> 21.8 mm
- net +3V3: track 141.7 -> 145.7 mm, vias 6 -> 8
- net Net-(J1-Pad4): track 0.00 -> 3.81 mm, vias 0 -> 1
- net Net-(J1-Pad3): track 3.64 -> 0.00 mm, vias 1 -> 0
- net Net-(Q2-Pad1): track 3.20 -> 0.00 mm
- net /SCL: track 6.34 -> 8.18 mm
- net Net-(Q1-Pad1): track 1.75 -> 0.00 mm
- net /SDA: track 8.50 -> 9.97 mm
- net GND: track 81.2 -> 81.3 mm, vias 4 -> 5
