File: hardware/mqtt_gateway/mqtt_gateway.kicad_pcb (KiCad board)
At the start: 4 copper layers, 75 x 51 mm, 64 parts, among them J1 awesome:RJ45-CAN, J2 Button-Sensors-MicroMatch2X03, J3 RJ45_Amphenol_RJMG1BD3B8K1ANR, J4 WAGO250-204, J5 Button-Sensors-MicroMatch2X03, U1 wuerthDebug6, U2 LD1117S33TR_SOT223, U3 PESD2CAN, U4 MCP2562-E-SN, U6 ESP32-WROOM-32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

Commit message: feat: Prepare mqtt gateway 3.0
Parts:
- removed C17: 100n, Capacitor_SMD:C_0402_1005Metric_Pad0.74x0.62mm_HandSolder
- removed R18: 10K, Resistor_SMD:R_0402_1005Metric_Pad0.72x0.64mm_HandSolder
- removed R7: 12K1 1%, Resistor_SMD:R_0603_1608Metric_Pad0.98x0.95mm_HandSolder
- removed U7: LAN8720A, Package_DFN_QFN:QFN-24-1EP_4x4mm_P0.5mm_EP2.6x2.6mm
- added C10: 22u, Capacitor_SMD:C_0805_2012Metric_Pad1.18x1.45mm_HandSolder, F.Cu at (106.4, 111.3)
- added C11: 100n, Capacitor_SMD:C_0603_1608Metric_Pad1.08x0.95mm_HandSolder, F.Cu at (108.2, 111.3)
- added R35: 10K, Resistor_SMD:R_0603_1608Metric_Pad0.98x0.95mm_HandSolder, F.Cu at (149.9, 98.3)
- added U5: KSZ8081MLX, Package_QFP:LQFP-48_7x7mm_P0.5mm, F.Cu at (115.2, 107.8)
- C14: value 470p -> 100n; footprint Capacitor_SMD:C_0402_1005Metric_Pad0.74x0.62mm_HandSolder -> Capacitor_SMD:C_0603_1608Metric_Pad1.08x0.95mm_HandSolder
- C15: value 1u -> 2u2; footprint Capacitor_SMD:C_0402_1005Metric_Pad0.74x0.62mm_HandSolder -> Capacitor_SMD:C_0603_1608Metric_Pad1.08x0.95mm_HandSolder
- C16: value 1u -> 22u; footprint Capacitor_SMD:C_0402_1005Metric_Pad0.74x0.62mm_HandSolder -> Capacitor_SMD:C_0805_2012Metric_Pad1.18x1.45mm_HandSolder
- C7, C8: footprint Capacitor_SMD:C_0402_1005Metric_Pad0.74x0.62mm_HandSolder -> Capacitor_SMD:C_0603_1608Metric_Pad1.08x0.95mm_HandSolder
- FB1: value Ferrite_Bead_Small -> BLM18KG331SH1D
- R10, R11: value 1K -> 220R
- R16, R2: footprint Resistor_SMD:R_0402_1005Metric_Pad0.72x0.64mm_HandSolder -> Resistor_SMD:R_0603_1608Metric_Pad0.98x0.95mm_HandSolder; moved to B.Cu
- R8, R9: value 10K -> 4K7
- moved R10 14.1 mm to (134.8, 91.9), turned to -90 degrees
- moved R9 14.1 mm to (134.8, 88.6)
- moved R28 10.7 mm to (107.4, 107.2), turned to 0 degrees
- moved C15 10.4 mm to (118.4, 100.2), turned to -90 degrees
- moved C7 10.4 mm to (119.9, 100.2)
- moved C14 7.83 mm to (115.2, 114.0)
- moved C8 4.76 mm to (115.9, 100.7), turned to 0 degrees
- moved C16 3.36 mm to (115.7, 98.9), turned to 180 degrees
- moved R8 3.35 mm to (113.4, 78.0), turned to -90 degrees
- moved R11 3.32 mm to (113.4, 81.3)
- moved FB1 2.50 mm to (118.6, 96.5)
- moved R2 1.53 mm to (113.1, 110.5), turned to 180 degrees
- moved R19 1.32 mm to (126.1, 100.1)
- moved R25 1.30 mm to (125.6, 113.7)
- moved R16 0.81 mm to (113.1, 108.7), turned to 180 degrees
Connections:
- C16 pad 1: VDDA -> GND
- C16 pad 2: GND -> VDDA
- C7 pad 1: VDDA -> GND
- C7 pad 2: GND -> Net-(C14-Pad2)
- J3 pad L1: Net-(J3-PadL1) -> Net-(J3-LEDY_A)
- J3 pad L2: Net-(J3-PadL2) -> Net-(J3-LEDY_K)
- J3 pad L3: Net-(J3-PadL3) -> Net-(J3-LEDG_K)
- J3 pad L4: Net-(J3-PadL4) -> Net-(J3-LEDG_A)
- R10 pad 1: Net-(J3-PadL3) -> +3.3V
- R10 pad 2: GND -> Net-(J3-LEDG_A)
- R11 pad 1: Net-(J3-PadL2) -> +3.3V
- R11 pad 2: GND -> Net-(J3-LEDY_A)
- R19 pad 1: Net-(R19-Pad1) -> Net-(U6-IO16)
- R8 pad 1: Net-(J3-PadL1) -> Net-(J3-LEDY_K)
- R8 pad 2: GND -> +3.3V
- R9 pad 1: Net-(J3-PadL4) -> Net-(J3-LEDG_K)
- R9 pad 2: GND -> +3.3V
- U6 pad 27: /B4-0 -> Net-(U6-IO16)
- U6 pad 28: Net-(R19-Pad1) -> /B4-0
Routing:
- net Net-(J3-LEDG_K): track 0.00 -> 76.5 mm, vias 0 -> 1
- net Net-(J3-LEDY_K): track 0.00 -> 55.9 mm, vias 0 -> 1
- net Net-(J3-PadL4): track 47.8 -> 0.00 mm, vias 2 -> 0
- net Net-(J3-PadL1): track 38.8 -> 0.00 mm, vias 1 -> 0
- net Net-(J3-LEDG_A): track 0.00 -> 18.6 mm
- net Net-(C14-Pad2): track 2.35 -> 16.7 mm, vias 0 -> 2
- net VDDA: track 52.4 -> 39.4 mm, vias 4 -> 2
- net Net-(J3-TD-): track 29.2 -> 37.6 mm
- net GND: track 99.9 -> 107.8 mm, vias 22 -> 20
- net Net-(J3-PadL2): track 6.97 -> 0.00 mm
- net Net-(J3-PadL3): track 6.79 -> 0.00 mm
- net /TXD0: track 12.1 -> 18.2 mm, vias 2 -> 0
- net Net-(J3-LEDY_A): track 0.00 -> 5.81 mm
- net /NRST: track 16.2 -> 10.5 mm, vias 2 -> 0
- net Net-(J3-TD+): track 39.4 -> 45.0 mm
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Other:
- board text added: "MQTT Gateway v2.0 2023-07-03"
- board text removed: "MQTT Gateway v1.0 2022-10-06"
